File: CESP.sch (KiCad schematic (older format))
At the start: 5 parts

Commit message: Version1 commit
Parts:
- removed U?: LTC1594CS, TSSOP14, symbol LTC1594CS
- removed U?: TL074, TSSOP14, symbol TL074
- removed U? (x3): TL074, symbol TL074
- added BT1: BATTERY, ~, symbol BATTERY
- added C1, C2: 100uF, ~, symbol CP1
- added D1, D2: LED, ~, symbol LED
- added Q1, Q2: NPN, ~, symbol NPN
- added R1, R4: 470, ~, symbol RESISTOR
- added R2, R3: 10k, ~, symbol RESISTOR
Connections:
- wire segments 0 -> 21
Other:
- note removed: "NOTE: THIS IS JUST A TEST BOARD\nREMOVE ALL COMPONENTS AND CREATE YOUR OWN\nINCLUDE SCHEMATIC HOOKUPS/NETLIST"
Changed lines of the file:
@@
-EESchema Schematic File Version 2  date 1/24/2014 12:04:40 AM
+EESchema Schematic File Version 2  date 1/26/2014 7:45:28 PM
 LIBS:power
 LIBS:device
@@
 LIBS:contrib
 LIBS:valves
+LIBS:accelerometer
+LIBS:GTB
+LIBS:LEDs
+LIBS:op-amp
+LIBS:redrawnDevice
+LIBS:Video
 LIBS:CESP-cache
 EELAYER 27 0
@@
 Sheet 1 1
 Title ""
-Date "24 jan 2014"
+Date "27 jan 2014"
 Rev ""
 Comp ""
@@
 $EndDescr
 $Comp
-L LTC1594CS U?
-U 1 1 52E1F38F
-P 3750 3300
-F 0 "U?" H 3750 3950 60  0000 C CNN
-F 1 "LTC1594CS" H 3750 2650 60  0000 C CNN
-F 2 "TSSOP14" H 3750 3300 60  0000 C CNN
-F 3 "" H 3750 3300 60  0000 C CNN
-	1    3750 3300
-	1    0    0    -1
-$EndComp
-$Comp
-L TL074 U?
-U 1 1 52E1F3CD
-P 7150 2150
-F 0 "U?" H 7200 2350 60  0000 C CNN
-F 1 "TL074" H 7300 1950 50  0000 C CNN
-F 2 "TSSOP14" H 7150 2150 60  0000 C CNN
-F 3 "" H 7150 2150 60  0000 C CNN
-	1    7150 2150
-	1    0    0    -1
-$EndComp
-$Comp
-L TL074 U?
-U 2 1 52E1F3DA
-P 7200 3500
-F 0 "U?" H 7250 3700 60  0000 C CNN
-F 1 "TL074" H 7350 3300 50  0000 C CNN
-F 2 "" H 7200 3500 60  0000 C CNN
-F 3 "" H 7200 3500 60  0000 C CNN
-	2    7200 3500
-	1    0    0    -1
-$EndComp
-$Comp
-L TL074 U?
-U 1 1 52E1F3E5
-P 8600 3500
-F 0 "U?" H 8650 3700 60  0000 C CNN
-F 1 "TL074" H 8750 3300 50  0000 C CNN
-F 2 "" H 8600 3500 60  0000 C CNN
-F 3 "" H 8600 3500 60  0000 C CNN
-	1    8600 3500
-	1    0    0    -1
-$EndComp
-$Comp
-L TL074 U?
-U 1 1 52E1F3EB
-P 8550 2100
-F 0 "U?" H 8600 2300 60  0000 C CNN
-F 1 "TL074" H 8700 1900 50  0000 C CNN
-F 2 "" H 8550 2100 60  0000 C CNN
-F 3 "" H 8550 2100 60  0000 C CNN
-	1    8550 2100
-	1    0    0    -1
-$EndComp
-Text Notes 4450 4650 0    80   ~ 0
-NOTE: THIS IS JUST A TEST BOARD\nREMOVE ALL COMPONENTS AND CREATE YOUR OWN\nINCLUDE SCHEMATIC HOOKUPS/NETLIST
+L NPN Q2
+U 1 1 52E59E7A
+P 6550 4200
+F 0 "Q2" H 6550 4050 50  0000 R CNN
+F 1 "NPN" H 6550 4350 50  0000 R CNN
+F 2 "~" H 6550 4200 60  0000 C CNN
+F 3 "~" H 6550 4200 60  0000 C CNN
+	1    6550 4200
+	1    0    0    -1
+$EndComp
+$Comp
+L NPN Q1
+U 1 1 52E59E87
+P 5000 4200
+F 0 "Q1" H 5000 4050 50  0000 R CNN
+F 1 "NPN" H 5000 4350 50  0000 R CNN
+F 2 "~" H 5000 4200 60  0000 C CNN
+F 3 "~" H 5000 4200 60  0000 C CNN
+	1    5000 4200
+	-1   0    0    -1
+$EndComp
+$Comp
+L RESISTOR R1
+U 1 1 52E59EDE
+P 4900 2725
+F 0 "R1" V 4800 2725 40  0000 C CNN
+F 1 "470" V 5000 2725 40  0000 C CNN
+F 2 "~" V 4830 2675 30  0000 C CNN
+F 3 "~" H 4900 2675 30  0000 C CNN
+	1    4900 2725
+	1    0    0    -1
+$EndComp
+$Comp
+L RESISTOR R2
+U 1 1 52E59EEB
+P 5550 2725
+F 0 "R2" V 5450 2725 40  0000 C CNN
+F 1 "10k" V 5650 2725 40  0000 C CNN
+F 2 "~" V 5480 2675 30  0000 C CNN
+F 3 "~" H 5550 2675 30  0000 C CNN
+	1    5550 2725
+	1    0    0    -1
+$EndComp
+$Comp
+L RESISTOR R4
+U 1 1 52E59F09
+P 6650 2725
+F 0 "R4" V 6550 2725 40  0000 C CNN
+F 1 "470" V 6750 2725 40  0000 C CNN
+F 2 "~" V 6580 2675 30  0000 C CNN
+F 3 "~" H 6650 2675 30  0000 C CNN
+	1    6650 2725
+	1    0    0    -1
+$EndComp
+$Comp
+L RESISTOR R3
+U 1 1 52E59F0F
+P 6050 2725
+F 0 "R3" V 5950 2725 40  0000 C CNN
+F 1 "10k" V 6150 2725 40  0000 C CNN
+F 2 "~" V 5980 2675 30  0000 C CNN
+F 3 "~" H 6050 2675 30  0000 C CNN
+	1    6050 2725
+	1    0    0    -1
+$EndComp
+$Comp
+L CP1 C2
+U 1 1 52E59F4A
+P 6375 3725
+F 0 "C2" H 6425 3825 50  0000 L CNN
+F 1 "100uF" H 6425 3625 50  0000 L CNN
+F 2 "~" H 6375 3725 60  0000 C CNN
+F 3 "~" H 6375 3725 60  0000 C CNN
+F 4 "399-6102-ND" H 6375 3725 60  0001 C CNN "digikey"
+	1    6375 3725
+	0    1    1    0
+$EndComp
+$Comp
+L CP1 C1
+U 1 1 52E59F71
+P 5125 3725
+F 0 "C1" H 5175 3825 50  0000 L CNN
+F 1 "100uF" H 5175 3625 50  0000 L CNN
+F 2 "~" H 5125 3725 60  0000 C CNN
+F 3 "~" H 5125 3725 60  0000 C CNN
+F 4 "399-6102-ND" H 5125 3725 60  0001 C CNN "Digikey"
+	1    5125 3725
+	0    -1   -1   0
+$EndComp
+$Comp
+L BATTERY BT1
+U 1 1 52E5A05A
+P 7275 3950
+F 0 "BT1" H 7275 4150 50  0000 C CNN
+F 1 "BATTERY" H 7275 3760 50  0000 C CNN
+F 2 "~" H 7275 3950 60  0000 C CNN
+F 3 "~" H 7275 3950 60  0000 C CNN
+	1    7275 3950
+	0    1    1    0
+$EndComp
+$Comp
+L LED D2
+U 1 1 52E5A0DB
+P 6650 3350
+F 0 "D2" H 6650 3450 50  0000 C CNN
+F 1 "LED" H 6650 3250 50  0000 C CNN
+F 2 "~" H 6650 3350 60  0000 C CNN
+F 3 "~" H 6650 3350 60  0000 C CNN
+	1    6650 3350
+	0    1    1    0
+$EndComp
+$Comp
+L LED D1
+U 1 1 52E5A0E8
+P 4900 3350
+F 0 "D1" H 4900 3450 50  0000 C CNN
+F 1 "LED" H 4900 3250 50  0000 C CNN
+F 2 "~" H 4900 3350 60  0000 C CNN
+F 3 "~" H 4900 3350 60  0000 C CNN
+	1    4900 3350
+	0    1    1    0
+$EndComp
+Wire Wire Line
+	5200 4200 5750 4200
+Wire Wire Line
+	5550 3000 5550 4200
+Wire Wire Line
+	6050 3000 6050 4200
+Wire Wire Line
+	5975 4200 6350 4200
+Wire Wire Line
+	6575 3725 6650 3725
+Connection ~ 6650 3725
+Wire Wire Line
+	5325 3725 5325 4025
+Wire Wire Line
+	5325 4025 5975 4025
+Wire Wire Line
+	5975 4025 5975 4200
+Connection ~ 6050 4200
+Wire Wire Line
+	6175 3725 5750 3725
+Wire Wire Line
+	5750 3725 5750 4200
+Connection ~ 5550 4200
+Wire Wire Line
+	4900 3725 4925 3725
+Connection ~ 4900 3725
+Wire Wire Line
+	4900 2500 7275 2500
+Connection ~ 5550 2500
+Connection ~ 6050 2500
+Wire Wire Line
+	4900 4400 4900 4550
+Wire Wire Line
+	4900 4550 7275 4550
+Wire Wire Line
+	6650 4550 6650 4400
+Wire Wire Line
+	7275 4550 7275 4250
+Connection ~ 6650 4550
+Wire Wire Line
+	7275 2500 7275 3650
+Connection ~ 6650 2500
+Wire Wire Line
+	4900 3000 4900 3150
+Wire Wire Line
+	4900 3550 4900 4000
+Wire Wire Line
+	6650 3550 6650 4000
+Wire Wire Line
+	6650 3000 6650 3150
 $EndSCHEMATC
